File: PCB/PCB.kicad_pcb (KiCad board)
At the start: 2 copper layers, 100 x 50 mm, 52 parts, among them J1 USB_C_Receptacle_USB2.0_16P, J2 18650, Q1 FS8205A, SW1 SW_Push_Reset, SW2 SW_Push_Boot, U1 HT-CT62, U2 SAM-M10Q, U3 ER_OLEDM0.91_1x-I2C, U4 TPS63001, U6 BQ24074RGT, U7 DW01A, U8 USBLC6-2SC6

Commit message: added BOM for stardance, fixed the j3, made it a connector, and re-exported gerbers
Parts:
- removed U3: ER_OLEDM0.91_1x-I2C, Display:ER_OLEDM0.91_1x-I2C
- added J3: OLED_0.91in_I2C, Connector_PinSocket_2.54mm:PinSocket_1x04_P2.54mm_Vertical, F.Cu at (144.0, 54.9)
- C6: value 10uf -> 10uF
- C8: value 0.1uF -> 100nF
- Q1: value FS8205A -> SI6968BEDQ
Routing:
- net GND: track 405.0 -> 406.7 mm
- net +3V3: track 185.1 -> 186.5 mm
- net OLED_SCL: track 20.8 -> 21.9 mm
