File: PCB/PCB.kicad_sch (KiCad schematic)
At the start: 50 parts, among them J1 USB_C_Receptacle_USB2.0_16P, J2 18650, Q1 FS8205A, SW1 SW_Push_Reset, SW2 SW_Push_Boot, U1 HT-CT62, U2 SAM-M10Q, U3 ER_OLEDM0.91_1x-I2C, U4 TPS63001, U6 BQ24074RGT, U7 DW01A, U8 USBLC6-2SC6

Commit message: started routing
Parts:
- J2: footprint Connector_JST:JST_PH_B2B-PH-K_1x02_P2.00mm_Vertical -> Battery:BatteryHolder_Keystone_1042_1x18650
Changed lines of the file:
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@@
 			)
 		)
-		(property "Footprint" "Connector_JST:JST_PH_B2B-PH-K_1x02_P2.00mm_Vertical"
+		(property "Footprint" "Battery:BatteryHolder_Keystone_1042_1x18650"
 			(at 80.01 92.71 0)
 			(hide yes)

Commit message: Fixed Bom again, made the oled DNP
Parts:
- C1: Manufacturer (none) -> Murata Electronics; Manufacturer Part # (none) -> GRT188R61H105KE13D
- C10, C12, C15, C2, C3, C5, C7: Manufacturer (none) -> Cal-Chip Electronics, Inc.; Manufacturer Part # (none) -> GMC21X7R106K25NT
- C11, C16, C18, C20, C21, C9: Manufacturer (none) -> Murata Electronics; Manufacturer Part # (none) -> GCJ188R71E104KA12D
- C13: Manufacturer (none) -> YAGEO; Manufacturer Part # (none) -> CC0603KRX5R8BB225
- C6: value 10uf -> 10uF; Manufacturer (none) -> Cal-Chip Electronics, Inc.; Manufacturer Part # (none) -> GMC21X7R106K25NT
- C8: value 0.1uF -> 100nF; Manufacturer (none) -> Murata Electronics; Manufacturer Part # (none) -> GCJ188R71E104KA12D
- D1: Manufacturer (none) -> Lite-On Inc.; Manufacturer Part # (none) -> LTST-C191KRKT
- F1: Manufacturer (none) -> Littelfuse Inc.; Manufacturer Part # (none) -> 1206L150SLYR
- J1: Manufacturer (none) -> Korean Hroparts Elec; Manufacturer Part # (none) -> TYPE-C-31-M-12
- J2: Manufacturer (none) -> Keystone Electronics; Manufacturer Part # (none) -> 1042
- L1: Manufacturer (none) -> Bourns Inc.; Manufacturer Part # (none) -> SRN3015-2R2M
- Q1: value FS8205A -> SI6968BEDQ; Manufacturer (none) -> Vishay Siliconix; Manufacturer Part # (none) -> SI6968BEDQ-T1-GE3
- R1, R2: Manufacturer (none) -> Bourns Inc.; Manufacturer Part # (none) -> CR0603-FX-5101ELF
- R10, R11, R19, TH1: Manufacturer (none) -> YAGEO; Manufacturer Part # (none) -> AR0603FR-0710KL
- R14, R15: Manufacturer (none) -> YAGEO; Manufacturer Part # (none) -> RC0603FR-07100KL
- R16: Manufacturer (none) -> YAGEO; Manufacturer Part # (none) -> RC0603FR-07470RL
- R17, R18: Manufacturer (none) -> YAGEO; Manufacturer Part # (none) -> RC0603FR-071KL
- R3, R4: Manufacturer (none) -> YAGEO; Manufacturer Part # (none) -> RC0603FR-0722RL
- R5: Manufacturer (none) -> YAGEO; Manufacturer Part # (none) -> RC0603FR-07100RL
- R6: Manufacturer (none) -> YAGEO; Manufacturer Part # (none) -> RC0603FR-073KL
- R7: Manufacturer (none) -> YAGEO; Manufacturer Part # (none) -> RC0603FR-073K09L
- R8, R9: Manufacturer (none) -> YAGEO; Manufacturer Part # (none) -> RC0603FR-074K7L
- SW1, SW2: Manufacturer (none) -> C&K; Manufacturer Part # (none) -> PTS810SJS250SMTR LFS
- U1: Comment (none) -> https://heltec.org/project/ht-ct62/ U1: HT-CT62 902–928 MHz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; Manufacturer (none) -> Heltec Automation; Manufacturer Part # (none) -> HT-CT62 902-928MHz
- U2: Manufacturer (none) -> u-blox; Manufacturer Part # (none) -> SAM-M10Q-00B
- U3: Comment (none) -> U3: DNP, customer will install.; now not fitted; now left out of the parts list
- U4: Manufacturer (none) -> Texas Instruments; Manufacturer Part # (none) -> TPS63001DRCR
- U6: Manufacturer (none) -> Texas Instruments; Manufacturer Part # (none) -> BQ24074RGTR
- U7: Manufacturer (none) -> Shenzhen Slkormicro Semicon Co., Ltd.; Manufacturer Part # (none) -> DW01A
- U8: Manufacturer (none) -> STMicroelectronics; Manufacturer Part # (none) -> USBLC6-2SC6

Commit message: added BOM for stardance, fixed the j3, made it a connector, and re-exported gerbers
Parts:
- removed U3: ER_OLEDM0.91_1x-I2C, Display:ER_OLEDM0.91_1x-I2C, symbol Display_Graphic:ER_OLEDM0.91_1x-I2C
- added J3: OLED_0.91in_I2C, Connector_PinSocket_2.54mm:PinSocket_1x04_P2.54mm_Vertical, symbol Connector:Conn_01x04_Socket
- F1: MPN 1206L150SLYR -> (none)
- Q1: value SI6968BEDQ -> SI6968BEDQ-T1-E3; MPN FS8205A -> (none); Manufacturer Vishay Siliconix -> Alpha & Omega Semiconductor Inc.; Manufacturer Part # SI6968BEDQ-T1-GE3 -> AO8814
- R10, R11, R19, TH1: Manufacturer Part # AR0603FR-0710KL -> AC0603FR-0710KL
- R14, R15: Manufacturer Part # RC0603FR-07100KL -> AR0603FR-07100KL
- R3, R4: Manufacturer YAGEO -> Panasonic Industry; Manufacturer Part # RC0603FR-0722RL -> ERJ-3EKF22R0V
- R5: Manufacturer Part # RC0603FR-07100RL -> AR0603FR-07100RL
- R8, R9: Manufacturer YAGEO -> Yageo
- U7: MPN DW01A -> (none)
Connections:
- net +3V3: now also J3.2 (Pin_2)
- net GND: now also J3.1 (Pin_1)
- net OLED_SCL: now also R9.2, J3.3 (Pin_3); no longer R8.2
- net OLED_SDA: now also R8.2, J3.4 (Pin_4); no longer R9.2
